Commit message: add objs to envs

File: diffusion_policy/env/franka_assembly/meshes/table/table.urdf (robot description, URDF)
Before this commit: robot table.urdf, 1 links, 0 joints
Links:
- added link cup, mass 0.1; collision cylinder length=0.08 radius=0.04; visual mesh filename=cup.stl scale=0.001 0.001 0.001
- added link pan, mass 0.3; collision cylinder length=0.02 radius=0.1; visual mesh filename=pan.stl scale=0.001 0.001 0.001
Joints:
- added joint cup_to_table: type fixed, parent baseLink, child cup, origin xyz=0 0 0.65 rpy=0 0 0
- added joint pan_to_table: type fixed, parent baseLink, child pan, origin xyz=0.2 0 0.63 rpy=0 0 0
